File: ProgrammerBoard/ProgrammerBoard.kicad_sch (KiCad schematic)
At the start: 0 parts

Commit message: 12345
Parts:
- added J1: 2 Position Terminal Block Header, rsx_headers_screw:CONN_1776508, symbol rsx_header_screw:2_Position_Terminal_Block_Header
Changed lines of the file:
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@@
 	(generator_version "10.0")
 	(paper "A4")
+	(symbol
+		(lib_id "rsx_header_screw:2_Position_Terminal_Block_Header")
+		(at 161.29 93.98 0)
+		(unit 1)
+		(body_style 1)
+		(exclude_from_sim no)
+		(in_bom yes)
+		(on_board yes)
+		(in_pos_files yes)
+		(dnp no)
+		(fields_autoplaced yes)
+		(property "Reference" "J1"
+			(at 163.83 95.2499 0)
+			(show_name no)
+			(do_not_autoplace no)
+			(effects
+				(font
+					(size 1.27 1.27)
+				)
+				(justify left)
+			)
+		)
+		(property "Value" "2 Position Terminal Block Header"
+			(at 161.29 99.06 0)
+			(hide yes)
+			(show_name no)
+			(do_not_autoplace no)
+			(effects
+				(font
+					(size 1.27 1.27)
+				)
+			)
+		)
+		(property "Footprint" "rsx_headers_screw:CONN_1776508"
+			(at 161.29 93.98 0)
+			(hide yes)
+			(show_name no)
+			(do_not_autoplace no)
+			(effects
+				(font
+					(size 1.27 1.27)
+				)
+			)
+		)
+		(property "Datasheet" "https://www.phoenixcontact.com/en-us/products/pcb-header-mstb-25-2-gf-508-1776508?type=pdf"
+			(at 161.29 93.98 0)
+			(hide yes)
+			(show_name no)
+			(do_not_autoplace no)
+			(effects
+				(font
+					(size 1.27 1.27)
+				)
+			)
+		)
+		(property "Description" "TERM BLOCK HDR 2POS 5.08MM"
+			(at 161.29 93.98 0)
+			(hide yes)
+			(show_name no)
+			(do_not_autoplace no)
+			(effects
+				(font
+					(size 1.27 1.27)
+				)
+			)
+		)
+		(property "MFR" "Phoenix Contact"
+			(at 161.29 93.98 0)
+			(hide yes)
+			(show_name no)
+			(do_not_autoplace no)
+			(effects
+				(font
+					(size 1.27 1.27)
+				)
+			)
+		)
+		(property "DPN" "277-5741-ND"
+			(at 161.29 93.98 0)
+			(hide yes)
+			(show_name no)
+			(do_not_autoplace no)
+			(effects
+				(font
+					(size 1.27 1.27)
+				)
+			)
+		)
+		(property "MPN" "1776508"
+			(at 161.29 93.98 0)
+			(hide yes)
+			(show_name no)
+			(do_not_autoplace no)
+			(effects
+				(font
+					(size 1.27 1.27)
+				)
+			)
+		)
+		(pin "1"
+		)
+		(pin "2"
+		)
+		(instances
+			(project "ProgrammerBoard"
+				(path "/eddff067-1d03-431d-9638-fe5f49ec946b"
+					(reference "J1")
+					(unit 1)
+				)
+			)
+		)
+	)
 	(sheet_instances
 		(path "/"

Commit message: Test
Parts:
- added U1: ATF1508ASx-xxJx84, Package_LCC:PLCC-84_29.3x29.3mm_P1.27mm, symbol CPLD_Microchip:ATF1508ASx-xxJx84
Connections:
- new net: U1.13 (VCCIO), U1.26 (VCCIO), U1.38 (VCCIO), U1.53 (VCCIO), U1.66 (VCCIO), U1.78 (VCCIO)
- new net: U1.19 (GND), U1.32 (GND), U1.42 (GND), U1.47 (GND), U1.59 (GND), U1.7 (GND), U1.72 (GND), U1.82 (GND)
- new net: U1.3 (VCCINT), U1.43 (VCCINT)
