File: ATMega/ATMega.kicad_sch (KiCad schematic)
At the start: 1 part, among them U1 ATmega328-P

Commit message: ATMega
- ATMega
Parts:
- removed U1: ATmega328-P, Package_DIP:DIP-28_W7.62mm, symbol MCU_Microchip_ATmega:ATmega328-P
- added ATMega328-20PU_Socket1: ic_conn_28pin, rsx_misc:OST_ED281DT, symbol rsx_misc:ic_conn_28pin
- added Arduino_TL_PowerPins1, Arduino_TR_DigitalPins1: Conn_01x06_Female, rsx_headers:PinSocket_1x06_P2.54mm_Vertical, symbol rsx_header:Conn_01x06_Female
- added Decoupling_Capacitor1, Decoupling_Capacitor2: 100n, Capacitor_SMD:C_0603_1608Metric, symbol rsx_Capacitors:100n
- added Electrolytic_Capacitor_Arduino1: 10u, rsx_capacitors:C_0805_2012Metric, symbol rsx_Capacitors:10u
- added R1: 10k, rsx_resistors:R_0603_1608Metric, symbol rsx_Resistors:10k
Connections:
- new net: Arduino_TR_DigitalPins1.1 (Pin_1), R1.2
- new net 5V: ATMega328-20PU_Socket1.20, ATMega328-20PU_Socket1.7, Arduino_TL_PowerPins1.4 (Pin_4), Decoupling_Capacitor1.1, Decoupling_Capacitor2.1
- new net Capacitor_Negative: Arduino_TL_PowerPins1.2 (Pin_2), Electrolytic_Capacitor_Arduino1.1
- new net Capacitor_Positive: Arduino_TL_PowerPins1.6 (Pin_6), Electrolytic_Capacitor_Arduino1.2
- new net GND: ATMega328-20PU_Socket1.22, ATMega328-20PU_Socket1.8, Arduino_TL_PowerPins1.3 (Pin_3), Decoupling_Capacitor1.2, Decoupling_Capacitor2.2
- new net MISO: ATMega328-20PU_Socket1.18, Arduino_TR_DigitalPins1.2 (Pin_2)
- new net MOSI: ATMega328-20PU_Socket1.17, Arduino_TR_DigitalPins1.3 (Pin_3)
- new net RESET: ATMega328-20PU_Socket1.1, Arduino_TR_DigitalPins1.4 (Pin_4)
- new net SCK: ATMega328-20PU_Socket1.19, R1.1
- no-connect marks 0 -> 24
Other:
- note added: "10"
- note added: "11"
- note added: "12"
- note added: "13"
- note added: "3.3V"
- note added: "5V"
- note added: "8"
- note added: "9"
- note added: "GND"
- note added: "RESET"
- note added: "VIN"

Commit message: ATMega adjust
Parts:
- removed Arduino_TL_PowerPins1, Arduino_TR_DigitalPins1: Conn_01x06_Female, rsx_headers:PinSocket_1x06_P2.54mm_Vertical, symbol rsx_header:Conn_01x06_Female
- removed R1: 10k, rsx_resistors:R_0603_1608Metric, symbol rsx_Resistors:10k
- added Arduino_BL1, Arduino_TR_2: header_1x6_arduino, Connector_PinHeader_2.54mm:PinHeader_1x06_P2.54mm_Vertical, symbol rsx_header:header_1x6_arduino
- added Arduino_BR1, Arduino_TL1: header_1x8_arduino, Connector_PinHeader_2.54mm:PinHeader_1x08_P2.54mm_Vertical, symbol rsx_header:header_1x8_arduino
- added Arduino_TR_1: header_1x4_arduino, Connector_PinHeader_2.54mm:PinHeader_1x04_P2.54mm_Vertical, symbol rsx_header:header_1x4_arduino
- added R2: 10k, rsx_resistors:R_0603_1608Metric, symbol rsx_Resistors:10k
Connections:
- net 5V: now also Arduino_TL1.4
- net Capacitor_Negative: now also Arduino_TL1.2
- net Capacitor_Positive: now also Arduino_TL1.6
- net GND: now also Arduino_TL1.3
- net MISO: now also Arduino_TR_2.2
- net MOSI: now also Arduino_TR_2.3
- net RESET: now also Arduino_TR_2.4
- net SCK: now also R2.1
- new net: Arduino_TR_2.1, R2.2
- no-connect marks 24 -> 44
Other:
- note added: "ANALOG PINS"
- note added: "DIGITAL PWM"
- note added: "IOREF"
- note added: "NC"
- note added: "~10"
- note added: "~11"
- note added: "~9"
- note removed: "10"
- note removed: "11"
- note removed: "9"
